File: PRO_MCU/PRO_MCU.kicad_sch (KiCad schematic)
At the start: 24 parts

Commit message: Updated KiCad project [After review]
Parts:
- removed R? (x2): 10K, Resistor_THT:R_Axial_DIN0207_L6.3mm_D2.5mm_P10.16mm_Horizontal, symbol Device:R
- R? (x2): value 470R -> 680R
Connections:
- net +BATT: now also U?.28 (VBAT); no longer U?.1 (P+), U?.3 (V+), U?.4 (VHI)
- net BL: now also U?.6 (A1); no longer U?.16 (RX_D0)
- net CS: now also U?.9 (A4); no longer U?.13 (MISO)
- net Display_RESET: now also U?.7 (A2); no longer U?.15 (TX_D1)
- net GND: now also U?.27 (GND); no longer U?.3 (EN)
- net Led_Red: now also U?.19 (D5_5V); no longer U?.23 (D11)
- net Pump_Ctrl: now also R?.1, R?.2
- net Sensor_RESET: now also U?.8 (A3); no longer U?.9 (A4)
- net Valve_Ctrl: now also U?.24 (D12); no longer R?.1, R?.2, U?.19 (D5_5V)
- new net VBUS: U?.1 (P+), U?.3 (V+), U?.4 (VHI)
Other:
- note added: "Connected to USART NC"
- note added: "D5 is 5V logic, used for red led"
- note added: "Internal 3v3 regulator, 3-5V in"
- note added: "led current limiting resistor integrated into button case"
- note removed: "D5 is 5V logic, used for 500mA pump"
- moved on the sheet: C?, D?, Q?, R?, U?

Commit message: Adds display EOC port
swaps some other pins around
Connections:
- net BL: now also U?.7 (A2); no longer U?.6 (A1)
- net Display_RESET: now also U?.8 (A3); no longer U?.7 (A2)
- net Sensor_RESET: now also U?.6 (A1); no longer U?.8 (A3)
- net Button_Red: now reaches C?.1, R?.1, R?.2, U?.21 (D9)
- net Button_Green: now reaches C?.1, R?.1, R?.2, U?.20 (D7)
- net EOC: now reaches U?.5 (A0)
Changed lines of the file:
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@@
+    (stroke (width 0) (type default) (color 0 0 0 0))
+  )
+  (polyline (pts (xy 223.52 57.15) (xy 223.52 90.17))
     (stroke (width 0) (type default) (color 0 0 0 0))
   )
@@
   )
   (wire (pts (xy 199.39 95.25) (xy 204.47 95.25))
+    (stroke (width 0) (type default) (color 0 0 0 0))
+  )
+  (polyline (pts (xy 223.52 57.15) (xy 259.08 57.15))
+    (stroke (width 0) (type default) (color 0 0 0 0))
+  )
+  (polyline (pts (xy 223.52 90.17) (xy 259.08 90.17))
+    (stroke (width 0) (type default) (color 0 0 0 0))
+  )
+  (polyline (pts (xy 259.08 90.17) (xy 259.08 57.15))
     (stroke (width 0) (type default) (color 0 0 0 0))
   )
@@
   )
   (text "led current limiting resistor integrated into button case"
-    (at 224.79 92.71 0)
+    (at 223.52 92.71 0)
     (effects (font (size 1.27 1.27)) (justify left bottom))
   )
@@
     (effects (font (size 1.27 1.27)) (justify left bottom))
   )
+  (label "Button_Green" (at 173.99 67.31 0)
+    (effects (font (size 1.27 1.27)) (justify left bottom))
+  )
+  (label "BL" (at 149.86 68.58 180)
+    (effects (font (size 1.27 1.27)) (justify right bottom))
+  )
+  (label "Display_RESET" (at 149.86 71.12 180)
+    (effects (font (size 1.27 1.27)) (justify right bottom))
+  )
   (label "Pump+" (at 33.02 39.37 0)
     (effects (font (size 1.27 1.27)) (justify left bottom))
@@
     (effects (font (size 1.27 1.27)) (justify left bottom))
   )
+  (label "EOC" (at 149.86 63.5 180)
+    (effects (font (size 1.27 1.27)) (justify right bottom))
+  )
   (label "MOSI" (at 231.14 137.16 180)
     (effects (font (size 1.27 1.27)) (justify right bottom))
@@
     (effects (font (size 1.27 1.27)) (justify right bottom))
   )
-  (label "Sensor_RESET" (at 149.86 71.12 180)
-    (effects (font (size 1.27 1.27)) (justify right bottom))
-  )
   (label "CS" (at 231.14 142.24 180)
     (effects (font (size 1.27 1.27)) (justify right bottom))
@@
     (effects (font (size 1.27 1.27)) (justify right bottom))
   )
+  (label "Button_Red" (at 173.99 69.85 0)
+    (effects (font (size 1.27 1.27)) (justify left bottom))
+  )
   (label "Valve-" (at 80.01 144.78 0)
     (effects (font (size 1.27 1.27)) (justify left bottom))
@@
     (effects (font (size 1.27 1.27)) (justify right bottom))
   )
-  (label "Display_RESET" (at 149.86 68.58 180)
-    (effects (font (size 1.27 1.27)) (justify right bottom))
-  )
   (label "Valve+" (at 33.02 41.91 0)
     (effects (font (size 1.27 1.27)) (justify left bottom))
@@
     (effects (font (size 1.27 1.27)) (justify right bottom))
   )
-  (label "BL" (at 149.86 66.04 180)
-    (effects (font (size 1.27 1.27)) (justify right bottom))
-  )
   (label "SCK" (at 231.14 139.7 180)
     (effects (font (size 1.27 1.27)) (justify right bottom))
@@
     (effects (font (size 1.27 1.27)) (justify left bottom))
   )
+  (label "Sensor_RESET" (at 149.86 66.04 180)
+    (effects (font (size 1.27 1.27)) (justify right bottom))
+  )
   (label "Led_Green" (at 173.99 72.39 0)

Commit message: Updates schematic symbols,, revised debouncing
- Updates electrical types of symbols in library
Parts:
- gave numbers to parts that had none: 22
Connections:
- net GND: now also Q1.1 (S), Q2.1 (S); no longer Q1.3 (S), Q2.3 (S)
- net Pump-: now also Q2.3 (D); no longer Q2.1 (D)
- net Valve-: now also Q1.3 (D); no longer Q1.1 (D)
- net VBUS renamed VDD
- no-connect marks 0 -> 10
Other:
- note added: "D2 should not be used due to crosstalk with the SPI flash."

Commit message: Updates project to KiCAD 7.0
Parts:
- removed R7, R8: 4K7, Resistor_THT:R_Axial_DIN0207_L6.3mm_D2.5mm_P10.16mm_Horizontal, symbol Device:R
- C2, C3, C4, C5: footprint (none) -> Capacitor_THT:C_Disc_D4.7mm_W2.5mm_P5.00mm
- D1, D2: footprint (none) -> LED_THT:LED_D3.0mm
- R5, R6: value 10K -> 4K7; now in the parts list
Connections:
- net +3.3V: no longer U4.2, U4.6 (2)
- net Button_Green: now also R5.1; no longer R5.2
- net Button_Red: now also R6.1; no longer R6.2
- net EOC: now also U3.6 (EOC)
- net GND: now also U4.2, U4.6 (2); no longer R5.1, R6.1
- net at U4.1: now also R5.2
- net at U4.5 (1): now also R6.2
- no-connect marks 10 -> 9
Other:
- note added: "Bounct nur ca. 50 us"
- note removed: "DNP"
- moved on the sheet: C2

Commit message: Updates layout, schematic, symbols and footprints
- Adds rounded corners to board geometry
- Component placement
- Modifications to schematic to make routing easier
Parts:
- C1: value 2u2 -> 4u7; footprint (none) -> Capacitor_SMD:C_0805_2012Metric_Pad1.18x1.45mm_HandSolder
- C2, C3, C4, C5: footprint Capacitor_THT:C_Disc_D4.7mm_W2.5mm_P5.00mm -> Capacitor_SMD:C_0805_2012Metric_Pad1.18x1.45mm_HandSolder
Connections:
- net EOC: now also U2.24 (D12); no longer U2.5 (A0)
- net Pump_Ctrl: now also U2.6 (A1); no longer U2.25 (D13)
- net Sensor_RESET: now also U2.25 (D13); no longer U2.6 (A1)
- net Valve_Ctrl: now also U2.5 (A0); no longer U2.24 (D12)
- no-connect marks 9 -> 8
Changed lines of the file:
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@@
   (no_connect (at 149.86 54.61))
   (no_connect (at 149.86 57.15))
-  (no_connect (at 173.99 74.93))
   (no_connect (at 173.99 44.45))
   (no_connect (at 173.99 57.15))
@@
     (effects (font (size 1.27 1.27)) (justify left bottom))
   )
-  (label "Pump_Ctrl" (at 173.99 80.01 0) (fields_autoplaced)
-    (effects (font (size 1.27 1.27)) (justify left bottom))
-  )
   (label "DC" (at 149.86 76.2 180) (fields_autoplaced)
     (effects (font (size 1.27 1.27)) (justify right bottom))
@@
     (effects (font (size 1.27 1.27)) (justify left bottom))
   )
-  (label "EOC" (at 149.86 63.5 180) (fields_autoplaced)
-    (effects (font (size 1.27 1.27)) (justify right bottom))
-  )
   (label "MOSI" (at 231.14 137.16 180) (fields_autoplaced)
     (effects (font (size 1.27 1.27)) (justify right bottom))
   )
+  (label "Valve_Ctrl" (at 149.86 63.5 180) (fields_autoplaced)
+    (effects (font (size 1.27 1.27)) (justify right bottom))
+  )
   (label "Display_RESET" (at 231.14 147.32 180) (fields_autoplaced)
     (effects (font (size 1.27 1.27)) (justify right bottom))
@@
     (effects (font (size 1.27 1.27)) (justify left bottom))
   )
+  (label "EOC" (at 173.99 77.47 0) (fields_autoplaced)
+    (effects (font (size 1.27 1.27)) (justify left bottom))
+  )
+  (label "Pump_Ctrl" (at 149.86 66.04 180) (fields_autoplaced)
+    (effects (font (size 1.27 1.27)) (justify right bottom))
+  )
   (label "Pump+" (at 140.97 140.97 0) (fields_autoplaced)
     (effects (font (size 1.27 1.27)) (justify left bottom))
@@
     (effects (font (size 1.27 1.27)) (justify left bottom))
   )
-  (label "Sensor_RESET" (at 149.86 66.04 180) (fields_autoplaced)
-    (effects (font (size 1.27 1.27)) (justify right bottom))
-  )
   (label "Led_Green" (at 173.99 72.39 0) (fields_autoplaced)
     (effects (font (size 1.27 1.27)) (justify left bottom))
   )
-  (label "Valve_Ctrl" (at 173.99 77.47 0) (fields_autoplaced)
-    (effects (font (size 1.27 1.27)) (justify left bottom))
+  (label "Sensor_RESET" (at 173.99 80.01 0) (fields_autoplaced)
+    (effects (font (size 1.27 1.27)) (justify left bottom))
+  )
+  (netclass_flag "" (length 2.54) (shape round) (at 148.59 39.37 0) (fields_autoplaced)
+    (effects (font (size 1.27 1.27)) (justify left bottom))
+    (property "Netclass" "Power" (at 149.2885 36.83 0)
+      (effects (font (size 1.27 1.27) italic) (justify left))
+    )
+  )
+  (netclass_flag "" (length 2.54) (shape round) (at 144.78 41.91 0) (fields_autoplaced)
+    (effects (font (size 1.27 1.27)) (justify left bottom))
+    (property "Netclass" "Power" (at 145.4785 39.37 0)
+      (effects (font (size 1.27 1.27) italic) (justify left))
+    )
+  )
+  (netclass_flag "" (length 2.54) (shape round) (at 137.16 44.45 0) (fields_autoplaced)
+    (effects (font (size 1.27 1.27)) (justify left bottom))
+    (property "Netclass" "Power" (at 137.8585 41.91 0)
+      (effects (font (size 1.27 1.27) italic) (justify left))
+    )
   )
   (symbol (lib_id "power:VDD") (at 140.97 34.29 0) (unit 1)
@@
       (effects (font (size 1.27 1.27)) (justify left))
     )
-    (property "Footprint" "Capacitor_THT:C_Disc_D4.7mm_W2.5mm_P5.00mm" (at 253.6952 40.64 0)
+    (property "Footprint" "Capacitor_SMD:C_0805_2012Metric_Pad1.18x1.45mm_HandSolder" (at 253.6952 40.64 0)
       (effects (font (size 1.27 1.27)) hide)
     )
@@
       (effects (font (size 1.27 1.27)) (justify left))
     )
-    (property "Footprint" "Capacitor_THT:C_Disc_D4.7mm_W2.5mm_P5.00mm" (at 200.3552 93.98 0)
+    (property "Footprint" "Capacitor_SMD:C_0805_2012Metric_Pad1.18x1.45mm_HandSolder" (at 200.3552 93.98 0)
       (effects (font (size 1.27 1.27)) hide)
     )
@@
       (effects (font (size 1.27 1.27)) (justify left))
     )
-    (property "Footprint" "Capacitor_THT:C_Disc_D4.7mm_W2.5mm_P5.00mm" (at 205.4352 139.7 0)
+    (property "Footprint" "Capacitor_SMD:C_0805_2012Metric_Pad1.18x1.45mm_HandSolder" (at 205.4352 139.7 0)
       (effects (font (size 1.27 1.27)) hide)
     )
@@
       (effects (font (size 1.27 1.27)) (justify left))
     )
-    (property "Value" "2u2" (at 114.3 43.1799 0)
-      (effects (font (size 1.27 1.27)) (justify left))
-    )
-    (property "Footprint" "" (at 111.4552 45.72 0)
+    (property "Value" "4u7" (at 114.3 43.1799 0)
+      (effects (font (size 1.27 1.27)) (justify left))
+    )
+    (property "Footprint" "Capacitor_SMD:C_0805_2012Metric_Pad1.18x1.45mm_HandSolder" (at 111.4552 45.72 0)
       (effects (font (size 1.27 1.27)) hide)
     )
@@
       (effects (font (size 1.27 1.27)) (justify left))
     )
-    (property "Footprint" "Capacitor_THT:C_Disc_D4.7mm_W2.5mm_P5.00mm" (at 200.3552 76.2 0)
-      (effects (font (size 1.27 1.27)) hide)
-    )
+    (property "Footprint" "Capacitor_SMD:C_0805_2012Metric_Pad1.18x1.45mm_HandSolder" (at 200.3552 76.2 0)
+      (effects (font (size 1.27 1.27)) hide)
+    )
