File: PRO_MCU/PRO_MCU.kicad_sch (KiCad schematic)
At the start: 20 parts, among them Q1 TN0702, Q2 TN0702, U1 Chassis, U2 ItsyBitsy_NRF52840, U3 MPRLS, U4 Buttons_LED, U5 waveshare_15867

Commit message: V1.0 Fabrication
Connections:
- net BL: now also U2.8 (A3); no longer U2.7 (A2)
- net CS: now also U2.10 (A5); no longer U2.9 (A4)
- net DC: now also U2.7 (A2); no longer U2.10 (A5)
- net Display_RESET: now also U2.9 (A4); no longer U2.8 (A3)
